File: NanoCompute/HDMI.kicad_sch (KiCad schematic)
At the start: 2 parts, among them J2 685119134923, J3 685119134923

Commit message: Added eMMC 5.1 HS400 128GB
It would act as a on-board primary storage while NVMe would act as an
extension/upgrade.
Other:
- title: Curiosity Board -> NanoCompute
Changed lines of the file:
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@@
 	(paper "A3")
 	(title_block
-		(title "Curiosity Board")
-		(date "2025-01-01")
+		(title "NanoCompute")
+		(date "2025-01-06")
 		(rev "v1.0")
 		(comment 3 "Power over Ethernet (PoE)")
@@
 		(pin "9"
 		)
-		(instances
-			(project ""
-				(path "/3a0a6fc3-d957-4804-b3c3-6d269c038b1f/61430c16-e72c-45ec-aff1-4e70bfe3da7d"
-					(reference "J2")
-					(unit 1)
-				)
-			)
-		)
-	)
+	)
