File: NanoCompute/LPDDR4.kicad_sch (KiCad schematic)
At the start: 2 parts, among them U2 MT53E1G32D2FW, U4 RK3588

Commit message: I think I added net classes(+coloring) for LPDDR4.
I'm not sure, it's 3AM I should check what I did tomorrow, figure our
those couple of signals that I don't understand where to connect or what
they are for. Probabbly could start working on the power section of the
LPDDR4. Need to check how much RAM will I actually need for 4K video
(@60fps?).
Connections:
- net DQ0_A: now also U4.U1 (DDR_CH0_DQ0_A); no longer U2.AA2 (DQ0_B)
- net DQ10_A: now also U4.AC1 (DDR_CH0_DQ10_A); no longer U2.V11 (DQ10_B)
- net DQ11_A: now also U4.AC2 (DDR_CH0_DQ11_A); no longer U2.U11 (DQ11_B)
- net DQ12_A: now also U4.Y1 (DDR_CH0_DQ12_A); no longer U2.U9 (DQ12_B)
- net DQ13_A: now also U4.Y2 (DDR_CH0_DQ13_A); no longer U2.V9 (DQ13_B)
- net DQ14_A: now also U4.AA1 (DDR_CH0_DQ14_A); no longer U2.Y9 (DQ14_B)
- net DQ15_A: now also U4.AA2 (DDR_CH0_DQ15_A); no longer U2.AA9 (DQ15_B)
- net DQ1_A: now also U4.T2 (DDR_CH0_DQ1_A); no longer U2.Y2 (DQ1_B)
- net DQ2_A: now also U4.T1 (DDR_CH0_DQ2_A); no longer U2.V2 (DQ2_B)
- net DQ3_A: now also U4.R2 (DDR_CH0_DQ3_A); no longer U2.U2 (DQ3_B)
- net DQ4_A: now also U4.W1 (DDR_CH0_DQ4_A); no longer U2.U4 (DQ4_B)
- net DQ5_A: now also U4.V2 (DDR_CH0_DQ5_A); no longer U2.V4 (DQ5_B)
- net DQ6_A: now also U4.V1 (DDR_CH0_DQ6_A); no longer U2.Y4 (DQ6_B)
- net DQ7_A: now also U4.U2 (DDR_CH0_DQ7_A); no longer U2.AA4 (DQ7_B)
- net DQ8_A: now also U4.AB2 (DDR_CH0_DQ8_A); no longer U2.AA11 (DQ8_B)
- net DQ9_A: now also U4.AB1 (DDR_CH0_DQ9_A); no longer U2.Y11 (DQ9_B)
- net DQ11_B: now reaches U4.B1 (DDR_CH0_DQ11_B)
- net DQ11_B: now also U2.U11 (DQ11_B)
- net DQ9_B: now reaches U4.C1 (DDR_CH0_DQ9_B)
- net DQ9_B: now also U2.Y11 (DQ9_B)
- net DQ10_B: now reaches U4.C2 (DDR_CH0_DQ10_B)
- net DQ10_B: now also U2.V11 (DQ10_B)
- net DQ15_B: now reaches U4.D1 (DDR_CH0_DQ15_B)
- net DQ15_B: now also U2.AA9 (DQ15_B)
- net DQ8_B: now reaches U4.D2 (DDR_CH0_DQ8_B)
- net DQ8_B: now also U2.AA11 (DQ8_B)
- net DQ13_B: now reaches U4.E1 (DDR_CH0_DQ13_B)
- net DQ13_B: now also U2.V9 (DQ13_B)
- net DQ14_B: now reaches U4.E2 (DDR_CH0_DQ14_B)
- net DQ14_B: now also U2.Y9 (DQ14_B)
- net DQ4_B: now reaches U4.F1 (DDR_CH0_DQ4_B)
- net DQ4_B: now also U2.U4 (DQ4_B)
- net DQ12_B: now reaches U4.F2 (DDR_CH0_DQ12_B)
- net DQ12_B: now also U2.U9 (DQ12_B)
- net DQ6_B: now reaches U4.G1 (DDR_CH0_DQ6_B)
- net DQ6_B: now also U2.Y4 (DQ6_B)
- net DQ5_B: now reaches U4.G2 (DDR_CH0_DQ5_B)
- net DQ5_B: now also U2.V4 (DQ5_B)
- net DQ0_B: now reaches U4.H1 (DDR_CH0_DQ0_B)
- net DQ0_B: now also U2.AA2 (DQ0_B)
- net DQ7_B: now reaches U4.H2 (DDR_CH0_DQ7_B)
- net DQ7_B: now also U2.AA4 (DQ7_B)
- net DQ2_B: now reaches U4.J1 (DDR_CH0_DQ2_B)
- net DQ2_B: now also U2.V2 (DQ2_B)
- net DQ1_B: now reaches U4.J2 (DDR_CH0_DQ1_B)
- net DQ1_B: now also U2.Y2 (DQ1_B)
- net DQ3_B: now reaches U4.K2 (DDR_CH0_DQ3_B)
- net DQ3_B: now also U2.U2 (DQ3_B)
- net CKE1_A: now reaches U4.N7 (DDR_CH0_LP4/4X_CKE1/LP5_CS1_A)
- net CKE1_A: now also U2.J5 (CKE1_A)
- net CA5_A: now reaches U4.P2 (DDR_CH0_A5_A)
- net CA5_A: now also U2.J11 (CA5_A)
- net CA2_A: now reaches U4.P4 (DDR_CH0_A2_A)
- net CA2_A: now also U2.H9 (CA2_A)
- net CA3_A: now reaches U4.P5 (DDR_CH0_A3_A)
- net CA3_A: now also U2.H10 (CA3_A)
- net CKE0_A: now reaches U4.P7 (DDR_CH0_LP4/4X_CKE0/LP5_CS0_A)
- net CKE0_A: now also U2.J4 (CKE0_A)
- net CA4_A: now reaches U4.R1 (DDR_CH0_A4_A)
- net CA4_A: now also U2.H11 (CA4_A)
- net CS0_A: now reaches U4.R6 (DDR_CH0_LP4/4X_CS0_A)
- net CS0_A: now also U2.H4 (CS0_A)
- net CS1_A: now reaches U4.R7 (DDR_CH0_LP4/4X_CS1_A)
- net CS1_A: now also U2.H3 (CS1_A)
- net CA0_A: now reaches U4.T7 (DDR_CH0_A0_A)
- net CA0_A: now also U2.H2 (CA0_A)
- net CA1_A: now reaches U4.T8 (DDR_CH0_A1_A)
- net CA1_A: now also U2.J2 (CA1_A)
- net DMI1_A: now reaches U2.C10 (DMI1_A)
- net DMIO_A: now reaches U2.C3 (DMI0_A)
- net CK_A_P: now reaches U2.J8 (CK_t_A)
- net CK_A_N: now reaches U2.J9 (CK_c_A)
Other:
- moved on the sheet: U2A, U2B, U2C, U4A

Commit message: Finished one LPDDR4 and connected it to LPDDR4 PHY
Connected the LPDDR4 to RK3588 LPDDR4 PHY, check all connections and it LGTM!
Added a second chip for additional 32Gb(4GB) LPDDR4 for total of 64Gb(8GB) of LPDRR4 memory.
Need to change nets for second chip from A->C and B->D.
Parts:
- added C5: 100n, Capacitor_SMD:C_0402_1005Metric, symbol Device:C_Small
- added R1, R13, R30, R31, R32, R34: 240R, Resistor_SMD:R_0402_1005Metric, symbol Device:R_Small_US
- added R33, R8: 10K, Resistor_SMD:R_0201_0603Metric, symbol Device:R_Small_US
- added unit 2 of U4
- added U9: MT53E1G32D2FW, CBFtLib:VFBGA200_10X14.5X1.1FW_MRN, symbol CBSymLib:MT53E1G32D2FW-046_IT_B
Connections:
- net CA0_A: now also U9.H2 (CA0_A)
- net CA1_A: now also U9.J2 (CA1_A)
- net CA2_A: now also U9.H9 (CA2_A)
- net CA3_A: now also U9.H10 (CA3_A)
- net CA4_A: now also U9.H11 (CA4_A)
- net CA5_A: now also U9.J11 (CA5_A)
- net CKE0_A: now also U9.J4 (CKE0_A)
- net CKE1_A: now also U9.J5 (CKE1_A)
- net CK_A_N: now also U2.P9 (CK_c_B), U4.M1 (DDR_CH0_CKB_B), U4.N1 (DDR_CH0_CKB_A), U9.J9 (CK_c_A), U9.P9 (CK_c_B)
- net CK_A_P: now also U2.P8 (CK_t_B), U4.M2 (DDR_CH0_CK_B), U4.N2 (DDR_CH0_CK_A), U9.J8 (CK_t_A), U9.P8 (CK_t_B)
- net CS0_A: now also U9.H4 (CS0_A)
- net CS1_A: now also U9.H3 (CS1_A)
- net DMI1_A: now also U4.AB4 (DDR_CH0_DM1_A), U9.C10 (DMI1_A)
- net DMIO_A: now also U4.Y4 (DDR_CH0_DM0_A), U9.C3 (DMI0_A)
- net DQ0_A: now also U9.B2 (DQ0_A)
- net DQ0_B: now also U9.AA2 (DQ0_B)
- net DQ10_A: now also U9.E11 (DQ10_A)
- net DQ10_B: now also U9.V11 (DQ10_B)
- net DQ11_A: now also U9.F11 (DQ11_A)
- net DQ11_B: now also U9.U11 (DQ11_B)
- net DQ12_A: now also U9.F9 (DQ12_A)
- net DQ12_B: now also U9.U9 (DQ12_B)
- net DQ13_A: now also U9.E9 (DQ13_A)
- net DQ13_B: now also U9.V9 (DQ13_B)
- net DQ14_A: now also U9.C9 (DQ14_A)
- net DQ14_B: now also U9.Y9 (DQ14_B)
- net DQ15_A: now also U9.B9 (DQ15_A)
- net DQ15_B: now also U9.AA9 (DQ15_B)
- net DQ1_A: now also U9.C2 (DQ1_A)
- net DQ1_B: now also U9.Y2 (DQ1_B)
- net DQ2_A: now also U9.E2 (DQ2_A)
- net DQ2_B: now also U9.V2 (DQ2_B)
- net DQ3_A: now also U9.F2 (DQ3_A)
- net DQ3_B: now also U9.U2 (DQ3_B)
- net DQ4_A: now also U9.F4 (DQ4_A)
- net DQ4_B: now also U9.U4 (DQ4_B)
- net DQ5_A: now also U9.E4 (DQ5_A)
- net DQ5_B: now also U9.V4 (DQ5_B)
- net DQ6_A: now also U9.C4 (DQ6_A)
- net DQ6_B: now also U9.Y4 (DQ6_B)
- net DQ7_A: now also U9.B4 (DQ7_A)
- net DQ7_B: now also U9.AA4 (DQ7_B)
- net DQ8_A: now also U9.B11 (DQ8_A)
- net DQ8_B: now also U9.AA11 (DQ8_B)
- net DQ9_A: now also U9.C11 (DQ9_A)
- net DQ9_B: now also U9.Y11 (DQ9_B)
- net GND: now also U4.M11 (DDR_CH0_PLL_AVSS), R30.2, R31.2, R33.2, R8.2
- net DQS1_A_N: now reaches U4.AA4 (DDR_CH0_DQS1N_A)
- net DQS1_A_N: now also U2.E10 (DQS1_c_A), U9.E10 (DQS1_c_A)
- net DQS1_A_P: now reaches U4.AA5 (DDR_CH0_DQS1P_A)
- net DQS1_A_P: now also U2.D10 (DQS1_t_A), U9.D10 (DQS1_t_A)
- net DMI1_B: now reaches U4.E4 (DDR_CH0_DM1_B)
- net DMI1_B: now also U2.Y10 (DMI1_B), U9.Y10 (DMI1_B)
- net DQS1_B_N: now reaches U4.F4 (DDR_CH0_DQS1N_B)
- net DQS1_B_N: now also U2.V10 (DQS1_c_B), U9.V10 (DQS1_c_B)
- net DQS1_B_P: now reaches U4.F5 (DDR_CH0_DQS1P_B)
- net DQS1_B_P: now also U2.W10 (DQS1_t_B), U9.W10 (DQS1_t_B)
- net DMIO_B: now reaches U4.G4 (DDR_CH0_DM0_B)
- net DMIO_B: now also U2.Y3 (DMI0_B), U9.Y3 (DMI0_B)
- net at U4.H7 (DDR_CH0_ZQ_B): now also R31.1
- net DQS0_B_N: now reaches U4.J7 (DDR_CH0_DQS0N_B)
- net DQS0_B_N: now also U2.V3 (DQS0_c_B), U9.V3 (DQS0_c_B)
- net DQS0_B_P: now reaches U4.J8 (DDR_CH0_DQS0P_B)
- net DQS0_B_P: now also U2.W3 (DQS0_t_B), U9.W3 (DQS0_t_B)
- net CA4_B: now reaches U4.K1 (DDR_CH0_A4_B)
- net CA4_B: now also U2.R11 (CA4_B), U9.R11 (CA4_B)
- net RESET_B: now reaches U4.K7 (DDR_CH0_RESET_B)
- net CA5_B: now reaches U4.L2 (DDR_CH0_A5_B)
- net CA5_B: now also U2.P11 (CA5_B), U9.P11 (CA5_B)
- net CKE1_B: now reaches U4.L4 (DDR_CH0_LP4/4X_CKE1/LP5_CS1_B)
- net CKE1_B: now also U2.P5 (CKE1_B), U9.P5 (CKE1_B)
- net CKE0_B: now reaches U4.L5 (DDR_CH0_LP4/4X_CKE0/LP5_CS0_B)
- net CKE0_B: now also U2.P4 (CKE0_B), U9.P4 (CKE0_B)
- net CS0_B: now reaches U4.L7 (DDR_CH0_LP4/4X_CS0_B)
- net CS0_B: now also U2.R4 (CS0_B), U9.R4 (CS0_B)
- net CS1_B: now reaches U4.L8 (DDR_CH0_LP4/4X_CS1_B)
- net CS1_B: now also U2.R3 (CS1_B), U9.R3 (CS1_B)
- net CA1_B: now reaches U4.M5 (DDR_CH0_A1_B)
- net CA1_B: now also U2.P2 (CA1_B), U9.P2 (CA1_B)
- net CA0_B: now reaches U4.M8 (DDR_CH0_A0_B)
- net CA0_B: now also U2.R2 (CA0_B), U9.R2 (CA0_B)
- net CA3_B: now reaches U4.N4 (DDR_CH0_A3_B)
- net CA3_B: now also U2.R10 (CA3_B), U9.R10 (CA3_B)
- net CA2_B: now reaches U4.N5 (DDR_CH0_A2_B)
- net CA2_B: now also U2.R9 (CA2_B), U9.R9 (CA2_B)
- net RESET_A: now reaches U4.T4 (DDR_CH0_RESET_A)
- net DQS0_A_N: now reaches U4.U4 (DDR_CH0_DQS0N_A)
- net DQS0_A_N: now also U2.E3 (DQS0_c_A), U9.E3 (DQS0_c_A)
- net DQS0_A_P: now reaches U4.U5 (DDR_CH0_DQS0P_A)
- net DQS0_A_P: now also U2.D3 (DQS0_t_A), U9.D3 (DQS0_t_A)
- net at U4.W8 (DDR_CH0_ZQ_A): now also R30.1
- net at U2.A5 (ZQ0): now also R13.2
- net at U2.A8 (ZQ1): now also R1.2
- net VDD2_DDR: now reaches U2.G2 (ODT_CA_A)
- net VDD2_DDR: now also U2.T2 (ODT_CA_B), R1.1, R13.1, R32.1, R34.1, U9.G2 (ODT_CA_A), U9.T2 (ODT_CA_B)
- net LPDDR4_RST_n: now reaches U2.T11 (RESET_n)
- net LPDDR4_RST_n: now also R33.1, R8.1, U9.T11 (RESET_n)
- new net: R34.2, U9.A5 (ZQ0)
- new net: R32.2, U9.A8 (ZQ1)
- no-connect marks 0 -> 10
Other:
- note added: "A -> C B -> D"
- moved on the sheet: U2A, U2B, U2C, U4A

Commit message: LPDDR4 second chip connected to LPDDR4 PHY
Added a missing Units for second LPDDR4 chip (VSS and Power).
Added a 1x100nF decoupling capacitor for each power rail of VDD1 but it
seems too much. Might need to find a better way of doing Low-Mid-High
range frequency decoupling.
Added TPS65296 as a LPddr4 Memory power solution but I need to check if
I can power both memory chips with just one TPS65296.
Parts:
- added C27, C28, C29, C30, C31, C32, C33, C34, C35, C36, C37, C38, C6, C7, C8: 100n, Capacitor_SMD:C_0402_1005Metric, symbol Device:C_Small
- added R35, R36: 240R, Resistor_SMD:R_0402_1005Metric, symbol Device:R_Small_US
- added unit 2 of U9
- added unit 3 of U9
Connections:
- net RESET_A is gone; now on net ~{RESET}_AB: U4.T4 (DDR_CH0_RESET_A)
- net CA0_A: no longer U9.H2 (CA0_A)
- net CA0_B: no longer U9.R2 (CA0_B)
- net CA1_A: no longer U9.J2 (CA1_A)
- net CA1_B: no longer U9.P2 (CA1_B)
- net CA2_A: no longer U9.H9 (CA2_A)
- net CA2_B: no longer U9.R9 (CA2_B)
- net CA3_A: no longer U9.H10 (CA3_A)
- net CA3_B: no longer U9.R10 (CA3_B)
- net CA4_A: no longer U9.H11 (CA4_A)
- net CA4_B: no longer U9.R11 (CA4_B)
- net CA5_A: no longer U9.J11 (CA5_A)
- net CA5_B: no longer U9.P11 (CA5_B)
- net CKE0_A: no longer U9.J4 (CKE0_A)
- net CKE0_B: no longer U9.P4 (CKE0_B)
- net CKE1_A: no longer U9.J5 (CKE1_A)
- net CKE1_B: no longer U9.P5 (CKE1_B)
- net CK_A_N: no longer U9.J9 (CK_c_A), U9.P9 (CK_c_B)
- net CK_A_P: no longer U9.J8 (CK_t_A), U9.P8 (CK_t_B)
- net CS0_A: no longer U9.H4 (CS0_A)
- net CS0_B: no longer U9.R4 (CS0_B)
- net CS1_A: no longer U9.H3 (CS1_A)
- net CS1_B: no longer U9.R3 (CS1_B)
- net DMI1_A: no longer U9.C10 (DMI1_A)
- net DMI1_B: no longer U9.Y10 (DMI1_B)
- net DMIO_A: no longer U9.C3 (DMI0_A)
- net DMIO_B: no longer U9.Y3 (DMI0_B)
- net DQ0_A: no longer U9.B2 (DQ0_A)
- net DQ0_B: no longer U9.AA2 (DQ0_B)
- net DQ10_A: no longer U9.E11 (DQ10_A)
- net DQ10_B: no longer U9.V11 (DQ10_B)
- net DQ11_A: no longer U9.F11 (DQ11_A)
- net DQ11_B: no longer U9.U11 (DQ11_B)
- net DQ12_A: no longer U9.F9 (DQ12_A)
- net DQ12_B: no longer U9.U9 (DQ12_B)
- net DQ13_A: no longer U9.E9 (DQ13_A)
- net DQ13_B: no longer U9.V9 (DQ13_B)
- net DQ14_A: no longer U9.C9 (DQ14_A)
- net DQ14_B: no longer U9.Y9 (DQ14_B)
- net DQ15_A: no longer U9.B9 (DQ15_A)
- net DQ15_B: no longer U9.AA9 (DQ15_B)
- net DQ1_A: no longer U9.C2 (DQ1_A)
- net DQ1_B: no longer U9.Y2 (DQ1_B)
- net DQ2_A: no longer U9.E2 (DQ2_A)
- net DQ2_B: no longer U9.V2 (DQ2_B)
- net DQ3_A: no longer U9.F2 (DQ3_A)
- net DQ3_B: no longer U9.U2 (DQ3_B)
- net DQ4_A: no longer U9.F4 (DQ4_A)
- net DQ4_B: no longer U9.U4 (DQ4_B)
- net DQ5_A: no longer U9.E4 (DQ5_A)
- net DQ5_B: no longer U9.V4 (DQ5_B)
- net DQ6_A: no longer U9.C4 (DQ6_A)
- net DQ6_B: no longer U9.Y4 (DQ6_B)
- net DQ7_A: no longer U9.B4 (DQ7_A)
- net DQ7_B: no longer U9.AA4 (DQ7_B)
- net DQ8_A: no longer U9.B11 (DQ8_A)
- net DQ8_B: no longer U9.AA11 (DQ8_B)
- net DQ9_A: no longer U9.C11 (DQ9_A)
- net DQ9_B: no longer U9.Y11 (DQ9_B)
- net DQS0_A_N: no longer U9.E3 (DQS0_c_A)
- net DQS0_A_P: no longer U9.D3 (DQS0_t_A)
- net DQS0_B_N: no longer U9.V3 (DQS0_c_B)
- net DQS0_B_P: no longer U9.W3 (DQS0_t_B)
- net DQS1_A_N: no longer U9.E10 (DQS1_c_A)
- net DQS1_A_P: no longer U9.D10 (DQS1_t_A)
- net DQS1_B_N: no longer U9.V10 (DQS1_c_B)
- net DQS1_B_P: no longer U9.W10 (DQS1_t_B)
- net GND: now also C5.2, U4.L16 (DDR_CH1_PLL_AVSS), C27.2, C28.2, C29.2, C30.2, C31.2, C32.2, C33.2, C34.2, C35.2, C36.2, C37.2, C38.2, C6.2, C7.2, C8.2, R35.2, R36.2, U9.A10 (VSS), U9.A3 (VSS), U9.AB10 (VSS), U9.AB3 (VSS), U9.AB5 (VSS), U9.AB8 (VSS), U9.C1 (VSS), U9.C12 (VSS), U9.C5 (VSS), U9.C8 (VSS), U9.D11 (VSS), U9.D2 (VSS), U9.D4 (VSS), U9.D9 (VSS), U9.E1 (VSS), U9.E12 (VSS), U9.E5 (VSS), U9.E8 (VSS), U9.G1 (VSS), U9.G10 (VSS), U9.G12 (VSS), U9.G3 (VSS), U9.G5 (VSS), U9.G8 (VSS), U9.J1 (VSS), U9.J10 (VSS), U9.J12 (VSS), U9.J3 (VSS), U9.K11 (VSS), U9.K2 (VSS), U9.K4 (VSS), U9.K9 (VSS), U9.N11 (VSS), U9.N2 (VSS), U9.N4 (VSS), U9.N9 (VSS), U9.P1 (VSS), U9.P10 (VSS), U9.P12 (VSS), U9.P3 (VSS), U9.T1 (VSS), U9.T10 (VSS), U9.T12 (VSS), U9.T3 (VSS), U9.T5 (VSS), U9.T8 (VSS), U9.V1 (VSS), U9.V12 (VSS), U9.V5 (VSS), U9.V8 (VSS), U9.W11 (VSS), U9.W2 (VSS), U9.W4 (VSS), U9.W9 (VSS), U9.Y1 (VSS), U9.Y12 (VSS), U9.Y5 (VSS), U9.Y8 (VSS)
- net VDD2_DDR: now also U2.A4 (VDD2), U2.A9 (VDD2), U2.AB4 (VDD2), U2.AB9 (VDD2), U2.F5 (VDD2), U2.F8 (VDD2), U2.H1 (VDD2), U2.H12 (VDD2), U2.H5 (VDD2), U2.H8 (VDD2), U2.K1 (VDD2), U2.K10 (VDD2), U2.K12 (VDD2), U2.K3 (VDD2), U2.N1 (VDD2), U2.N10 (VDD2), U2.N12 (VDD2), U2.N3 (VDD2), U2.R1 (VDD2), U2.R12 (VDD2), U2.R5 (VDD2), U2.R8 (VDD2), U2.U5 (VDD2), U2.U8 (VDD2), U9.A4 (VDD2), U9.A9 (VDD2), U9.AB4 (VDD2), U9.AB9 (VDD2), U9.F5 (VDD2), U9.F8 (VDD2), U9.H1 (VDD2), U9.H12 (VDD2), U9.H5 (VDD2), U9.H8 (VDD2), U9.K1 (VDD2), U9.K10 (VDD2), U9.K12 (VDD2), U9.K3 (VDD2), U9.N1 (VDD2), U9.N10 (VDD2), U9.N12 (VDD2), U9.N3 (VDD2), U9.R1 (VDD2), U9.R12 (VDD2), U9.R5 (VDD2), U9.R8 (VDD2), U9.U5 (VDD2), U9.U8 (VDD2)
- net CA4_C: now reaches U4.A10 (DDR_CH1_A4_C)
- net CA4_C: now also U9.H11 (CA4_A)
- net CK_C_N: now reaches U4.A12 (DDR_CH1_CKB_C)
- net CK_C_N: now also U9.J9 (CK_c_A)
- net CK_D_N: now reaches U4.A13 (DDR_CH1_CKB_D)
- net CK_D_N: now also U9.P9 (CK_c_B)
- net CA4_D: now reaches U4.A15 (DDR_CH1_A4_D)
- net CA4_D: now also U9.R11 (CA4_B)
- net DQ2_D: now reaches U4.A16 (DDR_CH1_DQ2_D)
- net DQ2_D: now also U9.V2 (DQ2_B)
- net DQ0_D: now reaches U4.A17 (DDR_CH1_DQ0_D)
- net DQ0_D: now also U9.AA2 (DQ0_B)
- net DQ6_D: now reaches U4.A18 (DDR_CH1_DQ6_D)
- net DQ6_D: now also U9.Y4 (DQ6_B)
- net DQ4_D: now reaches U4.A19 (DDR_CH1_DQ4_D)
- net DQ4_D: now also U9.U4 (DQ4_B)
- net DQ10_C: now reaches U4.A2 (DDR_CH1_DQ10_C)
- net DQ10_C: now also U9.E11 (DQ10_A)
- net DQ12_D: now reaches U4.A20 (DDR_CH1_DQ12_D)
- net DQ12_D: now also U9.U9 (DQ12_B)
- net DQ14_D: now reaches U4.A21 (DDR_CH1_DQ14_D)
- net DQ14_D: now also U9.Y9 (DQ14_B)
- net DQ8_D: now reaches U4.A22 (DDR_CH1_DQ8_D)
- net DQ8_D: now also U9.AA11 (DQ8_B)
- net DQ10_D: now reaches U4.A23 (DDR_CH1_DQ10_D)
- net DQ10_D: now also U9.V11 (DQ10_B)
- net DQ8_C: now reaches U4.A3 (DDR_CH1_DQ8_C)
- net DQ8_C: now also U9.B11 (DQ8_A)
- net DQ14_C: now reaches U4.A4 (DDR_CH1_DQ14_C)
- net DQ14_C: now also U9.C9 (DQ14_A)
- net DQ12_C: now reaches U4.A5 (DDR_CH1_DQ12_C)
- net DQ12_C: now also U9.F9 (DQ12_A)
- net DQ4_C: now reaches U4.A6 (DDR_CH1_DQ4_C)
- net DQ4_C: now also U9.F4 (DQ4_A)
- net DQ6_C: now reaches U4.A7 (DDR_CH1_DQ6_C)
- net DQ6_C: now also U9.C4 (DQ6_A)
- net DQ0_C: now reaches U4.A8 (DDR_CH1_DQ0_C)
- net DQ0_C: now also U9.B2 (DQ0_A)
- net DQ2_C: now reaches U4.A9 (DDR_CH1_DQ2_C)
- net DQ2_C: now also U9.E2 (DQ2_A)
- net DQ3_C: now reaches U4.B10 (DDR_CH1_DQ3_C)
- net DQ3_C: now also U9.F2 (DQ3_A)
- net CA5_C: now reaches U4.B11 (DDR_CH1_A5_C)
- net CA5_C: now also U9.J11 (CA5_A)
- net CK_C_P: now reaches U4.B12 (DDR_CH1_CK_C)
- net CK_C_P: now also U9.J8 (CK_t_A)
- net CK_D_P: now reaches U4.B13 (DDR_CH1_CK_D)
- net CK_D_P: now also U9.P8 (CK_t_B)
- net CA5_D: now reaches U4.B14 (DDR_CH1_A5_D)
- net CA5_D: now also U9.P11 (CA5_B)
- net DQ3_D: now reaches U4.B15 (DDR_CH1_DQ3_D)
- net DQ3_D: now also U9.U2 (DQ3_B)
- net DQ1_D: now reaches U4.B16 (DDR_CH1_DQ1_D)
- net DQ1_D: now also U9.Y2 (DQ1_B)
- net DQ7_D: now reaches U4.B17 (DDR_CH1_DQ7_D)
- net DQ7_D: now also U9.AA4 (DQ7_B)
- net DQ5_D: now reaches U4.B18 (DDR_CH1_DQ5_D)
- net DQ5_D: now also U9.V4 (DQ5_B)
- net DQ11_C: now reaches U4.B2 (DDR_CH1_DQ11_C)
- net DQ11_C: now also U9.F11 (DQ11_A)
- net DQ13_D: now reaches U4.B20 (DDR_CH1_DQ13_D)
- net DQ13_D: now also U9.V9 (DQ13_B)
- net DQ15_D: now reaches U4.B21 (DDR_CH1_DQ15_D)
- net DQ15_D: now also U9.AA9 (DQ15_B)
- net DQ9_D: now reaches U4.B22 (DDR_CH1_DQ9_D)
- net DQ9_D: now also U9.Y11 (DQ9_B)
- net DQ11_D: now reaches U4.B23 (DDR_CH1_DQ11_D)
- net DQ11_D: now also U9.U11 (DQ11_B)
- net DQ9_C: now reaches U4.B3 (DDR_CH1_DQ9_C)
- net DQ9_C: now also U9.C11 (DQ9_A)
- net DQ15_C: now reaches U4.B4 (DDR_CH1_DQ15_C)
- net DQ15_C: now also U9.B9 (DQ15_A)
- net DQ13_C: now reaches U4.B5 (DDR_CH1_DQ13_C)
- net DQ13_C: now also U9.E9 (DQ13_A)
- net DQ5_C: now reaches U4.B7 (DDR_CH1_DQ5_C)
- net DQ5_C: now also U9.E4 (DQ5_A)
- net DQ7_C: now reaches U4.B8 (DDR_CH1_DQ7_C)
- net DQ7_C: now also U9.B4 (DQ7_A)
- net DQ1_C: now reaches U4.B9 (DDR_CH1_DQ1_C)
- net DQ1_C: now also U9.C2 (DQ1_A)
- net CKE0_C: now reaches U4.D11 (DDR_CH1_LP4/4X_CKE0/LP5_CS0_C)
- net CKE0_C: now also U9.J4 (CKE0_A)
- net CA3_C: now reaches U4.D13 (DDR_CH1_A3_C)
- net CA3_C: now also U9.H10 (CA3_A)
- net CKE0_D: now reaches U4.D16 (DDR_CH1_LP4/4X_CKE0/LP5_CS0_D)
- net CKE0_D: now also U9.P4 (CKE0_B)
- net CS1_D: now reaches U4.D19 (DDR_CH1_LP4/4X_CS1_D)
- net CS1_D: now also U9.R3 (CS1_B)
- net DMIO_D: now reaches U4.D20 (DDR_CH1_DM0_D)
- net DMIO_D: now also U9.Y3 (DMI0_B)
- net DQS1_D_P: now reaches U4.D21 (DDR_CH1_DQS1P_D)
- net DQS1_D_P: now also U9.W10 (DQS1_t_B)
- net DMI1_D: now reaches U4.D22 (DDR_CH1_DM1_D)
- net DMI1_D: now also U9.Y10 (DMI1_B)
- net DMI1_C: now reaches U4.D4 (DDR_CH1_DM1_C)
- net DMI1_C: now also U9.C10 (DMI1_A)
- net DQS1_C_N: now reaches U4.D5 (DDR_CH1_DQS1N_C)
- net DQS1_C_N: now also U9.E10 (DQS1_c_A)
- net DQS0_C_N: now reaches U4.D9 (DDR_CH1_DQS0N_C)
- net DQS0_C_N: now also U9.E3 (DQS0_c_A)
- net ~{RESET}_CD: now reaches U4.E10 (DDR_CH1_RESET_C)
- net ~{RESET}_CD: now also R33.1, U9.T11 (RESET_n)
- net CKE1_C: now reaches U4.E11 (DDR_CH1_LP4/4X_CKE1/LP5_CS1_C)
- net CKE1_C: now also U9.J5 (CKE1_A)
- net CA2_C: now reaches U4.E13 (DDR_CH1_A2_C)
- net CA2_C: now also U9.H9 (CA2_A)
- net CA3_D: now reaches U4.E14 (DDR_CH1_A3_D)
- net CA3_D: now also U9.R10 (CA3_B)
- net CKE1_D: now reaches U4.E16 (DDR_CH1_LP4/4X_CKE1/LP5_CS1_D)
- net CKE1_D: now also U9.P5 (CKE1_B)
- net CS0_D: now reaches U4.E19 (DDR_CH1_LP4/4X_CS0_D)
- net CS0_D: now also U9.R4 (CS0_B)
- net DQS1_D_N: now reaches U4.E21 (DDR_CH1_DQS1N_D)
- net DQS1_D_N: now also U9.V10 (DQS1_c_B)
- net DQS1_C_P: now reaches U4.E5 (DDR_CH1_DQS1P_C)
- net DQS1_C_P: now also U9.D10 (DQS1_t_A)
- net DQS0_C_P: now reaches U4.E9 (DDR_CH1_DQS0P_C)
- net DQS0_C_P: now also U9.D3 (DQS0_t_A)
- net CA1_C: now reaches U4.F12 (DDR_CH1_A1_C)
- net CA1_C: now also U9.J2 (CA1_A)
- net at U4.F18 (DDR_CH1_ZQ_D): now also R36.1
- net DMIO_C: now reaches U4.F8 (DDR_CH1_DM0_C)
- net DMIO_C: now also U9.C3 (DMI0_A)
- net CS0_C: now reaches U4.G11 (DDR_CH1_LP4/4X_CS0_C)
- net CS0_C: now also U9.H4 (CS0_A)
- net CA0_C: now reaches U4.G12 (DDR_CH1_A0_C)
- net CA0_C: now also U9.H2 (CA0_A)
- net CA2_D: now reaches U4.G13 (DDR_CH1_A2_D)
- net CA2_D: now also U9.R9 (CA2_B)
- net CA1_D: now reaches U4.G14 (DDR_CH1_A1_D)
- net CA1_D: now also U9.P2 (CA1_B)
- net DQS0_D_N: now reaches U4.G16 (DDR_CH1_DQS0N_D)
- net DQS0_D_N: now also U9.V3 (DQS0_c_B)
- net at U4.G8 (DDR_CH1_ZQ_C): now also R35.1
- net CS1_C: now reaches U4.H11 (DDR_CH1_LP4/4X_CS1_C)
- net CS1_C: now also U9.H3 (CS1_A)
- net CA0_D: now reaches U4.H15 (DDR_CH1_A0_D)
- net CA0_D: now also U9.R2 (CA0_B)
- net DQS0_D_P: now reaches U4.H16 (DDR_CH1_DQS0P_D)
- net DQS0_D_P: now also U9.W3 (DQS0_t_B)
- net VDDQ_DDR: now reaches U2.AA10 (VDDQ)
- net VDDQ_DDR: now also U2.AA3 (VDDQ), U2.AA5 (VDDQ), U2.AA8 (VDDQ), U2.B10 (VDDQ), U2.B3 (VDDQ), U2.B5 (VDDQ), U2.B8 (VDDQ), U2.D1 (VDDQ), U2.D12 (VDDQ), U2.D5 (VDDQ), U2.D8 (VDDQ), U2.F10 (VDDQ), U2.F3 (VDDQ), U2.U10 (VDDQ), U2.U3 (VDDQ), U2.W1 (VDDQ), U2.W12 (VDDQ), U2.W5 (VDDQ), U2.W8 (VDDQ), U9.AA10 (VDDQ), U9.AA3 (VDDQ), U9.AA5 (VDDQ), U9.AA8 (VDDQ), U9.B10 (VDDQ), U9.B3 (VDDQ), U9.B5 (VDDQ), U9.B8 (VDDQ), U9.D1 (VDDQ), U9.D12 (VDDQ), U9.D5 (VDDQ), U9.D8 (VDDQ), U9.F10 (VDDQ), U9.F3 (VDDQ), U9.U10 (VDDQ), U9.U3 (VDDQ), U9.W1 (VDDQ), U9.W12 (VDDQ), U9.W5 (VDDQ), U9.W8 (VDDQ)
- net VCC1V8_DDR: now reaches U2.F1 (VDD1)
- net VCC1V8_DDR: now also C5.1, U2.F12 (VDD1), U2.G4 (VDD1), U2.G9 (VDD1), U2.T4 (VDD1), U2.T9 (VDD1), U2.U1 (VDD1), U2.U12 (VDD1), C27.1, C28.1, C29.1, C30.1, C31.1, C32.1, C33.1, C34.1, C35.1, C36.1, C37.1, C38.1, C6.1, C7.1, C8.1, U9.F1 (VDD1), U9.F12 (VDD1), U9.G4 (VDD1), U9.G9 (VDD1), U9.T4 (VDD1), U9.T9 (VDD1), U9.U1 (VDD1), U9.U12 (VDD1)
- net LPDDR4_RST_n renamed ~{RESET}_AB
- net ~{RESET}_AB: no longer R33.1, U9.T11 (RESET_n)
- net RESET_B: no longer names the net of U4.K7 (DDR_CH0_RESET_B)
- no-connect marks 10 -> 21
Other:
- note added: "Jesus, can I even put this on PCB?"
- note removed: "A -> C B -> D"
- moved on the sheet: C5, R1, R13, R30, R31, R32, R33, R34, R8, U2A, U2B, U2C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

Commit message: Added eMMC 5.1 HS400 128GB
It would act as a on-board primary storage while NVMe would act as an
extension/upgrade.
Other:
- title: CuriosityBoard -> NanoCompute
Changed lines of the file:
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@@
 	(paper "A2")
 	(title_block
-		(title "CuriosityBoard")
-		(date "2025-01-01")
+		(title "NanoCompute")
+		(date "2025-01-06")
 		(rev "v1.0")
 		(comment 4 "LPDDR4")
